Commit message: Add files via upload

File: urdf/hamster_bot_small.urdf (robot description, URDF)
Before this commit: robot my_mm_robot, 3 links, 2 joints
Links:
- link link_chassis: mass 1 -> 2; geometry collision box size=0.05 0.05 0.01; visual box size=0.05 0.05 0.01
- link link_left_wheel: mass 0.05 -> 0.5; geometry collision cylinder length=0.008 radius=${wheelRadius}; visual cylinder length=0.008 radius=${wheelRadius}
- link link_right_wheel: mass 0.05 -> 0.5; geometry collision cylinder length=0.008 radius=${wheelRadius}; visual cylinder length=0.008 radius=${wheelRadius}
Joints:
- joint joint_left_wheel: origin xyz=0.021 0.01 -0.002 rpy=0 0 0 -> xyz=0.04 0.0 -0.0 rpy=0 0 0
- joint joint_right_wheel: origin xyz=-0.021  0.01    -0.002 rpy=0 0 0 -> xyz=-0.04  0.0    -0.0 rpy=0 0 0
