Commit message: Add files via upload

File: urdf/hamster_bot.urdf (robot description, URDF)
Before this commit: robot my_mm_robot, 4 links, 3 joints
Links:
- removed link link_left_wheel
- removed link link_right_wheel
- removed link sensor_laser
- link link_chassis: mass 0.5 -> ${robot_mass}; geometry collision box size=0.04 0.01 0.01; visual box size=0.04 0.01 0.01
Joints:
- removed joint joint_sensor_laser
- joint joint_left_wheel: limit effort=5 velocity=6 -> effort=10 velocity=10; origin xyz=0.045 0.02 0 rpy=0 0 0 -> xyz=${-1*sphere_radius/2.0} 0.0 0.0 rpy=0 0 0
- joint joint_right_wheel: limit effort=5 velocity=6 -> effort=10 velocity=10; origin xyz=-0.045  0.02    0 rpy=0 0 0 -> xyz=${sphere_radius/2.0} 0.0 0.0 rpy=0 0 0
